File: HW/Solar_Array/Solar_Array.kicad_pcb (KiCad board)
At the start: 2 copper layers, 40 x 40 mm, 36 parts, among them J1 Conn_01x02, J3 Conn_01x02, J8 Conn_01x02, J9 Conn_01x02

Commit message: Fixed solar array copper pours and component links. Regenerated production data.
Parts:
- renumbered C10 to C1, C11 to C2, D21 to D1, D30 to D10, D31 to D11, D32 to D12, D33 to D13, D34 to D14, D35 to D15, D36 to D16, D22 to D2, D23 to D3, D24 to D4, D25 to D5, D26 to D6, D27 to D7, D28 to D8, D29 to D9, JP15 to JP1, JP24 to JP10, JP25 to JP11, JP26 to JP12, JP27 to JP13, JP28 to JP14, JP16 to JP2, JP17 to JP3, JP18 to JP4, JP19 to JP5, JP20 to JP6, JP21 to JP7, JP22 to JP8, JP23 to JP9
Connections:
- C1 pad 1: (no net) -> +PD
- C1 pad 2: (no net) -> GND
- C2 pad 1: (no net) -> +PD
- C2 pad 2: (no net) -> GND
- D1 pad 1: (no net) -> Net-(D1-K)
- D1 pad 2: (no net) -> Net-(D1-A)
- D10 pad 1: (no net) -> Net-(D10-K)
- D10 pad 2: (no net) -> Net-(D10-A)
- D11 pad 1: (no net) -> Net-(D11-K)
- D11 pad 2: (no net) -> Net-(D10-K)
- D12 pad 1: (no net) -> Net-(D12-K)
- D12 pad 2: (no net) -> Net-(D11-K)
- D13 pad 1: (no net) -> Net-(D13-K)
- D13 pad 2: (no net) -> Net-(D13-A)
- D14 pad 1: (no net) -> Net-(D14-K)
- D14 pad 2: (no net) -> Net-(D13-K)
- D15 pad 1: (no net) -> Net-(D15-K)
- D15 pad 2: (no net) -> Net-(D14-K)
- D16 pad 1: (no net) -> Net-(D16-K)
- D16 pad 2: (no net) -> Net-(D15-K)
- D2 pad 1: (no net) -> Net-(D2-K)
- D2 pad 2: (no net) -> Net-(D1-K)
- D3 pad 1: (no net) -> Net-(D3-K)
- D3 pad 2: (no net) -> Net-(D2-K)
- D4 pad 1: (no net) -> GND
- D4 pad 2: (no net) -> Net-(D3-K)
- D5 pad 1: (no net) -> Net-(D5-K)
- D5 pad 2: (no net) -> Net-(D5-A)
- D6 pad 1: (no net) -> Net-(D6-K)
- D6 pad 2: (no net) -> Net-(D5-K)
- D7 pad 1: (no net) -> Net-(D7-K)
- D7 pad 2: (no net) -> Net-(D6-K)
- D8 pad 1: (no net) -> Net-(D8-K)
- D8 pad 2: (no net) -> Net-(D7-K)
- D9 pad 1: (no net) -> Net-(D10-A)
- D9 pad 2: (no net) -> Net-(D9-A)
- J1 pad 1: (no net) -> +PD
- J1 pad 2: (no net) -> +PD
- J3 pad 1: (no net) -> GND
- J3 pad 2: (no net) -> GND
- J8 pad 1: (no net) -> +PD
- J8 pad 2: (no net) -> +PD
- J9 pad 1: (no net) -> GND
- J9 pad 2: (no net) -> GND
- JP1 pad 1: (no net) -> Net-(D1-A)
- JP1 pad 2: (no net) -> Net-(JP1-B)
- JP10 pad 1: (no net) -> Net-(D16-K)
- JP10 pad 2: (no net) -> Net-(D12-K)
- JP11 pad 1: (no net) -> GND
- JP11 pad 2: (no net) -> Net-(D12-K)
- JP12 pad 1: (no net) -> Net-(D16-K)
- JP12 pad 2: (no net) -> Net-(JP12-B)
- JP13 pad 1: (no net) -> +PD
- JP13 pad 2: (no net) -> Net-(JP12-B)
- JP14 pad 1: (no net) -> Net-(D13-A)
- JP14 pad 2: (no net) -> +PD
- JP2 pad 1: (no net) -> Net-(D8-K)
- JP2 pad 2: (no net) -> GND
- JP3 pad 1: (no net) -> Net-(D8-K)
- JP3 pad 2: (no net) -> Net-(JP1-B)
- JP4 pad 1: (no net) -> Net-(JP4-A)
- JP4 pad 2: (no net) -> Net-(JP1-B)
- JP5 pad 1: (no net) -> Net-(D5-A)
- JP5 pad 2: (no net) -> Net-(JP4-A)
- JP6 pad 1: (no net) -> Net-(D12-K)
- JP6 pad 2: (no net) -> Net-(D8-K)
- JP7 pad 1: (no net) -> Net-(D12-K)
- JP7 pad 2: (no net) -> Net-(JP4-A)
- JP8 pad 1: (no net) -> Net-(JP12-B)
- JP8 pad 2: (no net) -> Net-(JP4-A)
- JP9 pad 1: (no net) -> Net-(D9-A)
- JP9 pad 2: (no net) -> Net-(JP12-B)
Routing:
- net (no net): track 184.0 -> 0.00 mm
- net Net-(JP12-B): track 0.00 -> 26.6 mm
- net Net-(D8-K): track 0.00 -> 24.9 mm
- net Net-(D12-K): track 0.00 -> 22.6 mm
- net Net-(JP4-A): track 0.00 -> 21.4 mm
- net Net-(D16-K): track 0.00 -> 19.3 mm
- net Net-(JP1-B): track 0.00 -> 16.4 mm
- net Net-(D1-A): track 0.00 -> 4.21 mm
- net Net-(D7-K): track 0.00 -> 3.93 mm
- net Net-(D11-K): track 0.00 -> 3.93 mm
- net Net-(D3-K): track 0.00 -> 3.92 mm
- net Net-(D15-K): track 0.00 -> 3.92 mm
- net GND: track 0.00 -> 3.88 mm
- net +PD: track 0.00 -> 3.57 mm
- net Net-(D5-K): track 0.00 -> 3.43 mm
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- added copper zone on B.Cu, net +PD
- added copper zone on F.Cu, net +PD
- added copper zone on B.Cu, net GND
- added copper zone on F.Cu, net GND
- removed copper zone on B.Cu, net (none)
- removed copper zone on F.Cu, net (none)
