File: HW/Solar_Array/Solar_Array.kicad_sch (KiCad schematic)
At the start: 36 parts, among them J1 Conn_01x02, J2 Conn_01x02, J3 Conn_01x02, J4 Conn_01x02

Commit message: Fixed solar array copper pours and component links. Regenerated production data.
Parts:
- renumbered J4 to J3, J3 to J8, J2 to J9
Changed lines of the file:
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@@
 		(on_board yes)
 		(dnp no)
-		(property "Reference" "J3"
+		(property "Reference" "J8"
 			(at 252.222 85.09 0)
 			(effects
@@
 			(project "Solar_Array"
 				(path "/011c63e0-39e1-4fa5-83a2-f641a2cc657e"
-					(reference "J3")
+					(reference "J8")
 					(unit 1)
 				)
@@
 		(on_board yes)
 		(dnp no)
-		(property "Reference" "J2"
+		(property "Reference" "J9"
 			(at 241.3 100.076 0)
 			(effects
@@
 			(project "Solar_Array"
 				(path "/011c63e0-39e1-4fa5-83a2-f641a2cc657e"
-					(reference "J2")
+					(reference "J9")
 					(unit 1)
 				)
@@
 		(on_board yes)
 		(dnp no)
-		(property "Reference" "J4"
+		(property "Reference" "J3"
 			(at 252.222 100.33 0)
 			(effects
@@
 			(project "Solar_Array"
 				(path "/011c63e0-39e1-4fa5-83a2-f641a2cc657e"
-					(reference "J4")
-					(unit 1)
-				)
+					(reference "J3")
+					(unit 1)
+				)
